File: hardware/Victor9K_pga2350.kicad_pcb (KiCad board)
At the start: 4 copper layers, 232.7 x 126.4 mm, 28 parts, among them IC1 74LVC1G14GW,125, J1 PICO DEBUG, J2 Micro_SD_Card, J4 DX07S016JA1R1500, J5 UART, SW1 BOOTSEL, U1 ESP32-S3-DevKitC

Commit message: initial version of re-worked hardware removing the 74LVC245's
Parts:
- removed C14, C16, C17, C18, C9: 0.1µF, Capacitor_THT:C_Disc_D5.0mm_W2.5mm_P5.00mm
- removed C21: 10µF, Capacitor_THT:CP_Axial_L10.0mm_D4.5mm_P15.00mm_Horizontal
- added C2: 10µF, Capacitor_THT:C_Disc_D5.0mm_W2.5mm_P5.00mm, F.Cu at (160.4, 138.7)
- C10: value 0.1µF -> 10µF
- C3: value 10µF -> 0.1µF
- GF1: footprint Victor9000:Victor Gold Fingers 3 -> Victor9000:Victor_Gold_Fingers_3
- moved C11 203.7 mm to (120.8, 38.3)
- moved SW1 109.3 mm to (259.8, 93.5)
- moved C5 86.5 mm to (156.7, 97.2), turned to 0 degrees
- moved C4 86.5 mm to (160.8, 152.6), turned to 0 degrees
- moved C12 83.3 mm to (245.0, 123.4)
- moved C8 62.0 mm to (120.4, 87.8)
- moved C10 49.2 mm to (120.7, 35.0), turned to 180 degrees
- moved C7 42.2 mm to (120.3, 83.3), turned to 180 degrees
- moved C13 41.7 mm to (160.9, 91.2), turned to 180 degrees
- moved IC1 35.9 mm to (164.6, 90.5)
- moved C6 31.6 mm to (256.1, 141.8), turned to 180 degrees
- moved C1 23.1 mm to (140.7, 129.6)
- moved C3 22.2 mm to (140.7, 120.5)
- moved A1 19.3 mm to (163.0, 111.8)
- moved R2 5.06 mm to (257.3, 137.7)
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Connections:
- A1 pad 18: /PA17 -> /A17
- A1 pad 19: /PA18 -> /A18
- A1 pad 32: /IR_4 -> /IR4
- A1 pad 35: /IR_5 -> /IR5
- A1 pad 55: unconnected-(A1-3V3-Pad55) -> +3.3V
- C12 pad 1: +5V -> +3.3V
- C13 pad 1: +5V -> +3.3V
- C4 pad 1: +3.3V -> +5V
- C5 pad 1: +3.3V -> +5V
- C6 pad 1: +3.3V -> +5V
- C7 pad 1: +3.3V -> +5V
- C8 pad 1: +3.3V -> +5V
- GF1 pad 1: /A19 -> /A18
- GF1 pad 10: /READY -> /IO/M
- GF1 pad 11: /CLK15B -> /RD
- GF1 pad 12: GND -> /DT/R
- GF1 pad 13: /CLK5 -> /RESET
- GF1 pad 14: +5V -> /WR
- GF1 pad 15: +5V -> /NMI
- GF1 pad 16: GND -> /IRQ
- GF1 pad 17: /+12VLT -> /HOLD
- GF1 pad 18: /DLATCH -> /HLDA
- GF1 pad 19: /-12VLT -> /CSEN
- GF1 pad 2: /A17 -> /A16
- GF1 pad 20: GND -> /PHASE2
- GF1 pad 21: /EXTIO -> /XACK
- GF1 pad 22: /BD7 -> /BD6
- GF1 pad 23: /BD5 -> /BD4
- GF1 pad 24: /BD3 -> /BD2
- GF1 pad 25: /BD1 -> /BD0
- GF1 pad 26: /BD0 -> /BD1
- GF1 pad 27: /BD2 -> /BD3
- GF1 pad 28: /BD4 -> /BD5
- GF1 pad 29: /BD6 -> /BD7
- GF1 pad 3: /A15 -> /A14
- GF1 pad 30: /XACK -> /EXTIO
- GF1 pad 31: /PHASE2 -> GND
- GF1 pad 32: /CSEN -> /-12VLT
- GF1 pad 33: /HLDA -> /DLATCH
- GF1 pad 34: /HOLD -> /+12VLT
- GF1 pad 35: /IRQ -> GND
- GF1 pad 36: /NMI -> +5V
- GF1 pad 37: /WR -> +5V
- GF1 pad 38: /RESET -> /CLK5
- GF1 pad 39: /DT/R -> GND
- GF1 pad 4: /A13 -> /A12
- GF1 pad 40: /RD -> /CLK15B
- GF1 pad 41: /IO/M -> /READY
- GF1 pad 42: /ALE -> /IR5
- GF1 pad 43: /DEN -> /IR4
- GF1 pad 44: /SSO -> GND
- GF1 pad 45: /A8 -> /A9
- GF1 pad 46: /A10 -> /A11
- GF1 pad 47: /A12 -> /A13
- GF1 pad 48: /A14 -> /A15
- GF1 pad 49: /A16 -> /A17
- GF1 pad 5: /A11 -> /A10
- GF1 pad 50: /A18 -> /A19
- GF1 pad 6: /A9 -> /A8
- GF1 pad 7: GND -> /SSO
- GF1 pad 8: /IR4 -> /DEN
- GF1 pad 9: /IR5 -> /ALE
Routing:
- net +3.3V: track 0.00 -> 222.7 mm
- net /BD7: track 10.0 -> 127.9 mm
- net /BD6: track 13.5 -> 128.8 mm
- net /BD5: track 10.0 -> 123.7 mm, vias 0 -> 1
- net /BD4: track 13.5 -> 126.1 mm, vias 0 -> 1
- net /BD3: track 10.0 -> 120.8 mm, vias 0 -> 1
- net /BD2: track 13.5 -> 123.4 mm, vias 0 -> 1
- net /BD1: track 10.0 -> 118.5 mm, vias 0 -> 1
- net /BD0: track 13.5 -> 115.4 mm, vias 0 -> 1
- net +5V: track 175.3 -> 258.8 mm
- net /A19: track 10.0 -> 68.4 mm
- net /A17: track 10.0 -> 58.3 mm
- net /A18: track 13.5 -> 60.8 mm
- net /IR5: track 10.0 -> 57.0 mm
- net /A9: track 10.0 -> 53.1 mm, vias 0 -> 1
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